File: led-pov-board.kicad_pcb (KiCad board)
At the start: 2 copper layers, 300 x 30 mm, 18 parts, among them SW1 SW_Push, U1 ATtiny24A-SS

Commit message: add details to schematic
Parts:
- C1: value C_Small -> 1uF
- R1, R2, R3, R4, R5, R6, R7: value R -> 28 Ohm
Changed lines of the file:
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@@
         (effects (font (size 1 1) (thickness 0.15)))
     )
-    (fp_text value "C_Small" (at 0 -2.54) (layer "F.Fab") hide
+    (fp_text value "1uF" (at 0 -2.54) (layer "F.Fab") hide
         (effects (font (size 1 1) (thickness 0.15)))
     )
@@
         (effects (font (size 1 1) (thickness 0.15)))
     )
-    (fp_text value "R" (at 0 1.82) (layer "F.Fab") hide
+    (fp_text value "28 Ohm" (at 0 1.82) (layer "F.Fab") hide
         (effects (font (size 1 1) (thickness 0.15)))
     )
@@
         (effects (font (size 1 1) (thickness 0.15)))
     )
-    (fp_text value "R" (at 0 1.82) (layer "F.Fab") hide
+    (fp_text value "28 Ohm" (at 0 1.82) (layer "F.Fab") hide
         (effects (font (size 1 1) (thickness 0.15)))
     )
@@
         (effects (font (size 1 1) (thickness 0.15)))
     )
-    (fp_text value "R" (at 0 1.82) (layer "F.Fab") hide
+    (fp_text value "28 Ohm" (at 0 1.82) (layer "F.Fab") hide
         (effects (font (size 1 1) (thickness 0.15)))
     )
@@
         (effects (font (size 1 1) (thickness 0.15)))
     )
-    (fp_text value "R" (at 0 1.82) (layer "F.Fab") hide
+    (fp_text value "28 Ohm" (at 0 1.82) (layer "F.Fab") hide
         (effects (font (size 1 1) (thickness 0.15)))
     )
@@
         (effects (font (size 1 1) (thickness 0.15)))
     )
-    (fp_text value "R" (at 0 1.82) (layer "F.Fab") hide
+    (fp_text value "28 Ohm" (at 0 1.82) (layer "F.Fab") hide
         (effects (font (size 1 1) (thickness 0.15)))
     )
@@
         (effects (font (size 1 1) (thickness 0.15)))
     )
-    (fp_text value "R" (at 0 1.82) (layer "F.Fab") hide
+    (fp_text value "28 Ohm" (at 0 1.82) (layer "F.Fab") hide
         (effects (font (size 1 1) (thickness 0.15)))
     )
@@
         (effects (font (size 1 1) (thickness 0.15)))
     )
-    (fp_text value "R" (at 0 1.82) (layer "F.Fab") hide
-        (effects (font (size 1 1) (thickness 0.15)))
-    )
+    (fp_text value "28 Ohm" (at 0 1.82) (layer "F.Fab") hide
+        (effects (font (size 1 1) (thickness 0.15)))
+    )
